Commit message: added moveit generated package for the ur5 arm in the actual workcell

File: training/orig/demo_manipulation/robot_config/urdf/ur5_workspace.urdf (robot description, URDF)
Before this commit: robot ur5_workspace, 26 links, 25 joints
Links:
- removed link workcell_frame
- added link world_frame
- link gripper_body: geometry collision box size=0.044 0.088 0.0946; visual mesh filename=package://robot_config/meshes/vacuum_gripper_single_suction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
Joints:
- removed joint base_to_stand
- removed joint workcell_frame_to_cover_part1
- removed joint workcell_frame_to_cover_part2
- removed joint workcell_frame_to_front_wall2
- removed joint workcell_frame_to_left_wall2
- removed joint workcell_frame_to_right_wall2
- removed joint workcell_to_stand
- added joint stand_to_base: type fixed, parent ur5_stand, child base_link, origin xyz=0 0 0.1 rpy=0 0 2.355
- added joint world_frame_to_cover_part1: type fixed, parent world_frame, child cover_part1, origin xyz=-0.042 -0.081 0.07 rpy=0 0 0
- added joint world_frame_to_cover_part2: type fixed, parent world_frame, child cover_part2, origin xyz=-0.012 -0.465 0.07 rpy=0 0 0
- added joint world_frame_to_front_wall2: type fixed, parent world_frame, child front_wall2, origin xyz=-1.3375 0 0.5 rpy=0 0 0
- added joint world_frame_to_left_wall2: type fixed, parent world_frame, child left_wall2, origin xyz=-0.601 1.06 0.5 rpy=0 0 0
- added joint world_frame_to_right_wall2: type fixed, parent world_frame, child right_wall2, origin xyz=-0.601 -1.06 0.5 rpy=0 0 0
- added joint world_to_stand: type fixed, parent world_frame, child ur5_stand, origin xyz=-0.238 0 0.1
- joint elbow_joint: limit lower=-6.2831853 upper=6.2831853 effort=10.0 velocity=3.14159265 -> lower=-0.62831853 upper=2.827433385 effort=10.0 velocity=3.14159265
- joint shoulder_lift_joint: limit lower=-6.2831853 upper=6.2831853 effort=10.0 velocity=3.14159265 -> lower=-3.14159265 upper=3.14159265 effort=10.0 velocity=3.14159265
- joint shoulder_pan_joint: limit lower=-6.2831853 upper=6.2831853 effort=10.0 velocity=3.14159265 -> lower=-2.3561944875 upper=2.3561944875 effort=10.0 velocity=3.14159265
- joint to_gripper: child tcp_frame -> gripper_frame
- joint workcell_to_table_base2: parent workcell_frame -> world_frame
- joint wrist_1_joint: limit lower=-6.2831853 upper=6.2831853 effort=10.0 velocity=3.14159265 -> lower=-3.14159265 upper=0.0314159265 effort=10.0 velocity=3.14159265
- joint wrist_2_joint: limit lower=-6.2831853 upper=6.2831853 effort=10.0 velocity=3.14159265 -> lower=-3.14159265 upper=3.14159265 effort=10.0 velocity=3.14159265
- joint wrist_3_joint: limit lower=-6.2831853 upper=6.2831853 effort=10.0 velocity=3.14159265 -> lower=-4.712388975 upper=4.712388975 effort=10.0 velocity=3.14159265

File: training/orig/demo_manipulation/robot_config/urdf/ur5_workspace.xacro (robot description, xacro)
@@ -3,5 +3,5 @@
 	<include filename="$(find robot_config)/urdf/vacuum_gripper_macro.xacro"/>
 	<include filename="$(find ur5_description)/urdf/gazebo.urdf.xacro" />
-  	<include filename="$(find ur5_description)/urdf/model.urdf.xacro" />
+  	<include filename="$(find robot_config)/urdf/ur5_model.urdf.xacro" />
 	<include filename="$(find robot_config)/urdf/workspace_components.xacro"/>
 	<include filename="$(find robot_config)/urdf/kinect_sensor_macro.xacro"/>
