Commit message: finalized lesson 2.5 corrected lesson 2.6, 2.7

File: training/orig/2.6/lesson_tf_terminal/models/environment.xacro (robot description, xacro)
@@ -18,10 +18,10 @@
     <visual>
       <geometry>
-        <mesh filename="package://lesson_advanced_launch/models/grinder_visual.dae" />
+        <mesh filename="package://lesson_tf_terminal/models/grinder_visual.dae" />
       </geometry>
     </visual>
     <collision>
       <geometry>
-        <mesh filename="package://lesson_advanced_launch/models/grinder_collision.dae" />
+        <mesh filename="package://lesson_tf_terminal/models/grinder_collision.dae" />
       </geometry>
     </collision>

File: training/orig/2.6/lesson_tf_terminal/models/letterS.xacro (robot description, xacro)
@@ -6,5 +6,5 @@
 <!-- =================================================================================== -->
   <!-- This contains the macro "ses_part_macro" that places the clip wrt the tool tip -->
-  <include filename="$(find lesson_advanced_launch)/models/part.macro.xacro" />
+  <include filename="$(find lesson_tf_terminal)/models/part.macro.xacro" />
   <!-- Run the macro with the part name and offsets -->
   <xacro:ses_part_macro model_name="letterS.dae"

File: training/orig/2.6/lesson_tf_terminal/models/letterS_mount.xacro (robot description, xacro)
@@ -12,10 +12,10 @@
     <visual>
       <geometry>
-        <mesh filename="package://lesson_advanced_launch/models/letterS_mount_visual.dae" />
+        <mesh filename="package://lesson_tf_terminal/models/letterS_mount_visual.dae" />
       </geometry>>
     </visual>
     <collision>
       <geometry>
-        <mesh filename="package://lesson_advanced_launch/models/letterS_mount_collision.dae" />
+        <mesh filename="package://lesson_tf_terminal/models/letterS_mount_collision.dae" />
       </geometry>
     </collision>

File: training/orig/2.6/lesson_tf_terminal/models/part.macro.xacro (robot description, xacro)
@@ -14,10 +14,10 @@
     <visual>
       <geometry>
-        <mesh filename="package://lesson_advanced_launch/models/${model_name}" />
+        <mesh filename="package://lesson_tf_terminal/models/${model_name}" />
       </geometry>
     </visual>
     <collision>
       <geometry>
-        <mesh filename="package://lesson_advanced_launch/models/${model_name}" />
+        <mesh filename="package://lesson_tf_terminal/models/${model_name}" />
       </geometry>
     </collision>

File: training/orig/2.6/lesson_tf_terminal/models/puzzle_bent.xacro (robot description, xacro)
@@ -2,5 +2,5 @@
 <robot  xmlns:xacro="http://ros.org/wiki/xacro" name="part">
   <!-- This contains the macro "ses_part_macro" that places the clip wrt the tool tip -->
-  <include filename="$(find lesson_advanced_launch)/models/part.macro.xacro" />
+  <include filename="$(find lesson_tf_terminal)/models/part.macro.xacro" />
   <!-- Run the macro with the part name and offsets -->
   <xacro:ses_part_macro model_name="puzzle_bent.dae"

File: training/orig/2.6/lesson_tf_terminal/models/puzzle_flat.xacro (robot description, xacro)
@@ -2,5 +2,5 @@
 <robot  xmlns:xacro="http://ros.org/wiki/xacro" name="part">
   <!-- This contains the macro "ses_part_macro" that places the clip wrt the tool tip -->
-  <include filename="$(find lesson_advanced_launch)/models/part.macro.xacro" />
+  <include filename="$(find lesson_tf_terminal)/models/part.macro.xacro" />
   <!-- Run the macro with the part name and offsets -->
   <xacro:ses_part_macro model_name="puzzle_flat.dae"
@@ -11,9 +11,3 @@
                         model_rp="-0.2618"
                         model_ry="0" />
-                        <!--model_x="0.0110"
-                        model_y="0.0030"
-                        model_z="0.0315"
-                        model_rr="0"
-                        model_rp="-0.2618"
-                        model_ry="0" /-->
 </robot>

File: training/orig/2.6/lesson_tf_terminal/models/puzzle_mount_sia20.xacro (robot description, xacro)
@@ -12,10 +12,10 @@
     <visual>
       <geometry>
-        <mesh filename="package://lesson_advanced_launch/models/puzzle_mount_sia20_visual.stl" />
+        <mesh filename="package://lesson_tf_terminal/models/puzzle_mount_sia20_visual.stl" />
       </geometry>>
     </visual>
     <collision>
       <geometry>
-        <mesh filename="package://lesson_advanced_launch/models/puzzle_mount_sia20_collision.dae" />
+        <mesh filename="package://lesson_tf_terminal/models/puzzle_mount_sia20_collision.dae" />
       </geometry>
     </collision>

File: training/orig/2.7/lesson_tf_cpp/models/environment.xacro (robot description, xacro)
@@ -18,10 +18,10 @@
     <visual>
       <geometry>
-        <mesh filename="package://lesson_advanced_launch/models/grinder_visual.dae" />
+        <mesh filename="package://lesson_tf_cpp/models/grinder_visual.dae" />
       </geometry>
     </visual>
     <collision>
       <geometry>
-        <mesh filename="package://lesson_advanced_launch/models/grinder_collision.dae" />
+        <mesh filename="package://lesson_tf_cpp/models/grinder_collision.dae" />
       </geometry>
     </collision>

File: training/orig/2.7/lesson_tf_cpp/models/letterS.xacro (robot description, xacro)
@@ -6,5 +6,5 @@
 <!-- =================================================================================== -->
   <!-- This contains the macro "ses_part_macro" that places the clip wrt the tool tip -->
-  <include filename="$(find lesson_advanced_launch)/models/part.macro.xacro" />
+  <include filename="$(find lesson_tf_cpp)/models/part.macro.xacro" />
   <!-- Run the macro with the part name and offsets -->
   <xacro:ses_part_macro model_name="letterS.dae"

File: training/orig/2.7/lesson_tf_cpp/models/letterS_mount.xacro (robot description, xacro)
@@ -6,5 +6,5 @@
     <parent link="tool0" />
     <child link="ee_base" />
-    <origin xyz="0 0 0" rpy="0 0 0" />
+    <origin xyz="0.0127 0 0" rpy="0 0 0" />
   </joint>
   <!-- link "ee_base" and connected joints-->
@@ -12,10 +12,10 @@
     <visual>
       <geometry>
-        <mesh filename="package://lesson_tf_terminal/models/puzzle_mount_visual.dae" />
+        <mesh filename="package://lesson_tf_cpp/models/letterS_mount_visual.dae" />
       </geometry>>
     </visual>
     <collision>
       <geometry>
-        <mesh filename="package://lesson_tf_terminal/models/puzzle_mount_collision.dae" />
+        <mesh filename="package://lesson_tf_cpp/models/letterS_mount_collision.dae" />
       </geometry>
     </collision>
@@ -26,5 +26,5 @@
     <parent link="ee_base" />
     <child link="tool1" />
-    <origin xyz="0.0381 0.0 -0.011" rpy="${-150*deg} 0 ${90*deg}" />
+    <origin xyz="0.0680 -0.0032 0" rpy="${30*deg} ${90*deg} ${-90*deg}" />
   </joint>
 </robot>

File: training/orig/2.7/lesson_tf_cpp/models/part.macro.xacro (robot description, xacro)
@@ -14,10 +14,10 @@
     <visual>
       <geometry>
-        <mesh filename="package://lesson_advanced_launch/models/${model_name}" />
+        <mesh filename="package://lesson_tf_cpp/models/${model_name}" />
       </geometry>
     </visual>
     <collision>
       <geometry>
-        <mesh filename="package://lesson_advanced_launch/models/${model_name}" />
+        <mesh filename="package://lesson_tf_cpp/models/${model_name}" />
       </geometry>
     </collision>

File: training/orig/2.7/lesson_tf_cpp/models/puzzle_bent.xacro (robot description, xacro)
@@ -2,5 +2,5 @@
 <robot  xmlns:xacro="http://ros.org/wiki/xacro" name="part">
   <!-- This contains the macro "ses_part_macro" that places the clip wrt the tool tip -->
-  <include filename="$(find lesson_advanced_launch)/models/part.macro.xacro" />
+  <include filename="$(find lesson_tf_cpp)/models/part.macro.xacro" />
   <!-- Run the macro with the part name and offsets -->
   <xacro:ses_part_macro model_name="puzzle_bent.dae"

File: training/orig/2.7/lesson_tf_cpp/models/puzzle_flat.xacro (robot description, xacro)
@@ -2,5 +2,5 @@
 <robot  xmlns:xacro="http://ros.org/wiki/xacro" name="part">
   <!-- This contains the macro "ses_part_macro" that places the clip wrt the tool tip -->
-  <include filename="$(find lesson_advanced_launch)/models/part.macro.xacro" />
+  <include filename="$(find lesson_tf_cpp)/models/part.macro.xacro" />
   <!-- Run the macro with the part name and offsets -->
   <xacro:ses_part_macro model_name="puzzle_flat.dae"
@@ -11,9 +11,3 @@
                         model_rp="-0.2618"
                         model_ry="0" />
-                        <!--model_x="0.0110"
-                        model_y="0.0030"
-                        model_z="0.0315"
-                        model_rr="0"
-                        model_rp="-0.2618"
-                        model_ry="0" /-->
 </robot>

File: training/orig/2.7/lesson_tf_cpp/models/puzzle_mount.xacro (robot description, xacro)
@@ -12,10 +12,10 @@
     <visual>
       <geometry>
-        <mesh filename="package://lesson_advanced_launch/models/puzzle_mount_visual.dae" />
+        <mesh filename="package://lesson_tf_cpp/models/puzzle_mount_visual.dae" />
       </geometry>>
     </visual>
     <collision>
       <geometry>
-        <mesh filename="package://lesson_advanced_launch/models/puzzle_mount_collision.dae" />
+        <mesh filename="package://lesson_tf_cpp/models/puzzle_mount_collision.dae" />
       </geometry>
     </collision>

File: training/orig/2.7/lesson_tf_cpp/models/puzzle_mount_sia20.xacro (robot description, xacro)
@@ -12,10 +12,10 @@
     <visual>
       <geometry>
-        <mesh filename="package://lesson_advanced_launch/models/puzzle_mount_sia20_visual.stl" />
+        <mesh filename="package://lesson_tf_cpp/models/puzzle_mount_sia20_visual.stl" />
       </geometry>>
     </visual>
     <collision>
       <geometry>
-        <mesh filename="package://lesson_advanced_launch/models/puzzle_mount_sia20_collision.dae" />
+        <mesh filename="package://lesson_tf_cpp/models/puzzle_mount_sia20_collision.dae" />
       </geometry>
     </collision>

File: training/ref/2.6/lesson_tf_terminal/models/puzzle_mount.xacro (robot description, xacro)
@@ -12,10 +12,10 @@
     <visual>
       <geometry>
-        <mesh filename="package://lesson_advanced_launch/models/puzzle_mount_visual.dae" />
+        <mesh filename="package://lesson_tf_terminal/models/puzzle_mount_visual.dae" />
       </geometry>>
     </visual>
     <collision>
       <geometry>
-        <mesh filename="package://lesson_advanced_launch/models/puzzle_mount_collision.dae" />
+        <mesh filename="package://lesson_tf_terminal/models/puzzle_mount_collision.dae" />
       </geometry>
     </collision>
