Commit message: finished lessons 2.8 and 2.9

File: training/orig/2.8/lesson_urdf/urdf/sia20d_workspace.xacro (robot description, xacro)
@@ -1,3 +1,50 @@
 <?xml version="1.0" ?>
 <robot name="sia20d_workspace" xmlns:xacro="http://ros.org/wiki/xacro">
+	<include filename="$(find motoman_config)/cfg/sia20d_mesh_macro.xacro"/>
+	<include filename="$(find xacro_properties)/color_palette.xacro"/>  <!--contains colors used in this xacro-->
+	<include filename="$(find lesson_urdf)/urdf/vacuum_gripper_macro.xacro"/>
+	<include filename="$(find lesson_urdf)/urdf/workspace_components.xacro"/>
+	<include filename="$(find lesson_urdf)/urdf/kinect_sensor_macro.xacro"/>
+	<!-- property list -->
+	<xacro:property name="workcell_height" value="1"/>
+	<xacro:property name="coupler_height" value="0.087"/>
+	<!-- instantiating workcell definitions -->
+	<xacro:workcell_zone1_components/>
+	<!-- instantiating sensor definitions -->
+	<xacro:sensor_definitions parent_link="base_link" x_val="1.010" y_val="0.169" z_val="1.206" roll="0.005" pitch="1.968" yaw="0.0"/>
+	<!-- instantiating arm and gripper -->
+	<xacro:vacuum_gripper_definition gripper_adjustment="-0.01"/>
+	<xacro:sia20d_mesh prefix=""/>
+	<!-- arm-workcell joint definitions -->
+	<joint name="world_to_base" type="fixed">
+		<parent link="world_frame"/>
+		<child link="base_link"/>
+		<origin xyz="0.241 0 0" rpy="0 0 0"/>
+	</joint>
+	<!-- arm-gripper coupling link definitions-->
+	<link name="coupler">
+		<visual>
+			<geometry>
+				<mesh filename="package://lesson_urdf/meshes/COUPLER_visual.stl" />
+			</geometry>
+			<material name="orange"/>
+		</visual>
+		<collision>
+			<geometry>
+				<mesh filename="package://lesson_urdf/meshes/COUPLER_collision.stl" />
+			</geometry>
+			<material name="yellow"/>
+		</collision>
+	</link>
+	<!-- arm-gripper coupling joint definitions -->
+	<joint name="wrist_to_coupler" type="fixed">
+		<parent link="link_t"/>
+		<child link="coupler"/>
+		<origin xyz="0 0 0" rpy="1.570 0 -0.785"/>
+	</joint>
+	<joint name="coupler_to_gripper" type="fixed">
+		<parent link="coupler"/>
+		<child link="gripper_frame"/>
+		<origin xyz="0 ${coupler_height} 0" rpy="-1.570 3.14 0"/>
+	</joint>
 </robot>

File: training/orig/2.8/lesson_urdf/urdf/vacuum_gripper_macro.xacro (robot description, xacro)
@@ -1,3 +1,40 @@
 <?xml version="1.0" ?>
 <robot xmlns:xacro="http://ros.org/wiki/xacro">
+	<!-- parameter list -->
+	<xacro:property name="gripper_length" value="0.044"/>
+	<xacro:property name="gripper_width" value="0.088"/>
+	<xacro:property name="gripper_height" value="0.0946"/>
+	<xacro:macro name="vacuum_gripper_definition" params="gripper_adjustment">
+		<link name="gripper_frame"/>
+		<link name="gripper_body">
+			<visual>
+				<origin xyz="0 0 -0.048" rpy="0 0 0"/>
+				<geometry>
+					<mesh filename="package://lesson_urdf/meshes/vacuum_gripper_single_suction_cup.STL" />
+				</geometry>
+				<material name="silver">
+					<color rgba="0.8 0.8 0.8 1"/>
+				</material>
+			</visual>
+			<collision>
+				<geometry>
+					<box size="${gripper_length} ${gripper_width} ${gripper_height}"/>
+				</geometry>
+				<material name="another_blue2">
+					<color rgba="0.38 0.54 0.83 1"/>
+				</material>
+			</collision>
+		</link>
+		<link name="tcp_frame"/>
+		<joint name="gripper_to_palm" type="fixed">
+			<parent link="gripper_frame"/>
+			<child link="gripper_body"/>
+			<origin xyz="0 0 ${gripper_height * 0.5}" rpy="0 0 0"/>
+		</joint>
+		<joint name="gripper_to_tcp" type="fixed">
+			<parent link="gripper_frame"/>
+			<child link="tcp_frame"/>
+			<origin xyz=" 0 ${gripper_length * 0.5} ${0.12 + gripper_adjustment}" rpy="0 0 0"/>
+		</joint>
+	</xacro:macro>
 </robot>

File: training/orig/2.9/lesson_debug/models/environment.xacro (robot description, xacro)
@@ -18,10 +18,10 @@
     <visual>
       <geometry>
-        <mesh filename="package://lesson_advanced_launch/models/grinder_visual.dae" />
+        <mesh filename="package://lesson_debug/models/grinder_visual.dae" />
       </geometry>
     </visual>
     <collision>
       <geometry>
-        <mesh filename="package://lesson_advanced_launch/models/grinder_collision.dae" />
+        <mesh filename="package://lesson_debug/models/grinder_collision.dae" />
       </geometry>
     </collision>

File: training/orig/2.9/lesson_debug/models/letterS.xacro (robot description, xacro)
@@ -6,5 +6,5 @@
 <!-- =================================================================================== -->
   <!-- This contains the macro "ses_part_macro" that places the clip wrt the tool tip -->
-  <include filename="$(find lesson_advanced_launch)/models/part.macro.xacro" />
+  <include filename="$(find lesson_debug)/models/part.macro.xacro" />
   <!-- Run the macro with the part name and offsets -->
   <xacro:ses_part_macro model_name="letterS.dae"

File: training/orig/2.9/lesson_debug/models/letterS_mount.xacro (robot description, xacro)
@@ -6,5 +6,5 @@
     <parent link="tool0" />
     <child link="ee_base" />
-    <origin xyz="0 0 0" rpy="0 0 0" />
+    <origin xyz="0.0127 0 0" rpy="0 0 0" />
   </joint>
   <!-- link "ee_base" and connected joints-->
@@ -12,10 +12,10 @@
     <visual>
       <geometry>
-        <mesh filename="package://lesson_debug/models/puzzle_mount_visual.dae" />
+        <mesh filename="package://lesson_debug/models/letterS_mount_visual.dae" />
       </geometry>>
     </visual>
     <collision>
       <geometry>
-        <mesh filename="package://lesson_debug/models/puzzle_mount_collision.dae" />
+        <mesh filename="package://lesson_debug/models/letterS_mount_collision.dae" />
       </geometry>
     </collision>
@@ -26,5 +26,5 @@
     <parent link="ee_base" />
     <child link="tool1" />
-    <origin xyz="0.0381 0.0 -0.011" rpy="${-150*deg} 0 ${90*deg}" />
+    <origin xyz="0.0680 -0.0032 0" rpy="${30*deg} ${90*deg} ${-90*deg}" />
   </joint>
 </robot>

File: training/orig/2.9/lesson_debug/models/part.macro.xacro (robot description, xacro)
@@ -14,10 +14,10 @@
     <visual>
       <geometry>
-        <mesh filename="package://lesson_advanced_launch/models/${model_name}" />
+        <mesh filename="package://lesson_debug/models/${model_name}" />
       </geometry>
     </visual>
     <collision>
       <geometry>
-        <mesh filename="package://lesson_advanced_launch/models/${model_name}" />
+        <mesh filename="package://lesson_debug/models/${model_name}" />
       </geometry>
     </collision>

File: training/orig/2.9/lesson_debug/models/puzzle_bent.xacro (robot description, xacro)
@@ -2,5 +2,5 @@
 <robot  xmlns:xacro="http://ros.org/wiki/xacro" name="part">
   <!-- This contains the macro "ses_part_macro" that places the clip wrt the tool tip -->
-  <include filename="$(find lesson_advanced_launch)/models/part.macro.xacro" />
+  <include filename="$(find lesson_debug)/models/part.macro.xacro" />
   <!-- Run the macro with the part name and offsets -->
   <xacro:ses_part_macro model_name="puzzle_bent.dae"

File: training/orig/2.9/lesson_debug/models/puzzle_flat.xacro (robot description, xacro)
@@ -2,5 +2,5 @@
 <robot  xmlns:xacro="http://ros.org/wiki/xacro" name="part">
   <!-- This contains the macro "ses_part_macro" that places the clip wrt the tool tip -->
-  <include filename="$(find lesson_advanced_launch)/models/part.macro.xacro" />
+  <include filename="$(find lesson_debug)/models/part.macro.xacro" />
   <!-- Run the macro with the part name and offsets -->
   <xacro:ses_part_macro model_name="puzzle_flat.dae"
@@ -11,9 +11,3 @@
                         model_rp="-0.2618"
                         model_ry="0" />
-                        <!--model_x="0.0110"
-                        model_y="0.0030"
-                        model_z="0.0315"
-                        model_rr="0"
-                        model_rp="-0.2618"
-                        model_ry="0" /-->
 </robot>

File: training/orig/2.9/lesson_debug/models/puzzle_mount_sia20.xacro (robot description, xacro)
@@ -12,10 +12,10 @@
     <visual>
       <geometry>
-        <mesh filename="package://lesson_advanced_launch/models/puzzle_mount_sia20_visual.stl" />
+        <mesh filename="package://lesson_debug/models/puzzle_mount_sia20_visual.stl" />
       </geometry>>
     </visual>
     <collision>
       <geometry>
-        <mesh filename="package://lesson_advanced_launch/models/puzzle_mount_sia20_collision.dae" />
+        <mesh filename="package://lesson_debug/models/puzzle_mount_sia20_collision.dae" />
       </geometry>
     </collision>

File: training/ref/2.8/lesson_urdf/urdf/sia20d_workspace.xacro (robot description, xacro)
@@ -17,5 +17,5 @@
 	<xacro:sia20d_mesh prefix=""/>
 	<!-- arm-workcell joint definitions -->
-	<joint name="wordl_to_base" type="fixed">
+	<joint name="world_to_base" type="fixed">
 		<parent link="world_frame"/>
 		<child link="base_link"/>

File: training/ref/2.9/lesson_debug/models/puzzle_mount.xacro (robot description, xacro)
@@ -12,10 +12,10 @@
     <visual>
       <geometry>
-        <mesh filename="package://lesson_advanced_launch/models/puzzle_mount_visual.dae" />
+        <mesh filename="package://lesson_debug/models/puzzle_mount_visual.dae" />
       </geometry>>
     </visual>
     <collision>
       <geometry>
-        <mesh filename="package://lesson_advanced_launch/models/puzzle_mount_collision.dae" />
+        <mesh filename="package://lesson_debug/models/puzzle_mount_collision.dae" />
       </geometry>
     </collision>
